Commit message: added world link

File: boxer_description/urdf/boxer.urdf.xacro (robot description, xacro)
@@ -2,4 +2,5 @@
 <robot name="boxer" xmlns:xacro="http://www.ros.org/wiki/xacro">
   <xacro:include filename="$(find boxer_description)/urdf/materials.urdf.xacro"/>
+  <link name="world" />
   <!-- The robot's origin, center-bottom of the main chassis -->
   <link name="base_link" />

Commit message: reverted temporary changes

File: boxer_description/urdf/boxer.urdf.xacro (robot description, xacro)
@@ -2,5 +2,4 @@
 <robot name="boxer" xmlns:xacro="http://www.ros.org/wiki/xacro">
   <xacro:include filename="$(find boxer_description)/urdf/materials.urdf.xacro"/>
-  <link name="world" />
   <!-- The robot's origin, center-bottom of the main chassis -->
   <link name="base_link" />
